File: Isolated_supply_5V_15W.kicad_sch (KiCad schematic)
At the start: 26 parts, among them U25 LM5576

Commit message: Keyed stepper drivers. Larger input connector
Parts:
- renumbered C42 to C43, C43 to C44, C44 to C45, C45 to C46, C46 to C47, C47 to C48, C48 to C49, C49 to C50, C50 to C51, C51 to C52, C52 to C53, C53 to C54, C54 to C55, C55 to C56, C56 to C57, C57 to C58
Changed lines of the file:
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@@
   (symbol (lib_id "Device:C") (at 191.77 83.82 0) (unit 1)
     (in_bom yes) (on_board yes)
-    (property "Reference" "C51" (id 0) (at 193.04 81.2799 0)
+    (property "Reference" "C52" (id 0) (at 193.04 81.2799 0)
       (effects (font (size 1.27 1.27)) (justify left))
     )
@@
   (symbol (lib_id "Device:C") (at 148.59 74.93 0) (unit 1)
     (in_bom yes) (on_board yes)
-    (property "Reference" "C48" (id 0) (at 149.86 72.3899 0)
+    (property "Reference" "C49" (id 0) (at 149.86 72.3899 0)
       (effects (font (size 1.27 1.27)) (justify left))
     )
@@
   (symbol (lib_id "Device:C") (at 234.95 83.82 0) (unit 1)
     (in_bom yes) (on_board yes)
-    (property "Reference" "C55" (id 0) (at 236.22 81.28 0)
+    (property "Reference" "C56" (id 0) (at 236.22 81.28 0)
       (effects (font (size 1.27 1.27)) (justify left))
     )
@@
   (symbol (lib_id "Device:C") (at 162.56 83.82 0) (unit 1)
     (in_bom yes) (on_board yes)
-    (property "Reference" "C49" (id 0) (at 157.48 86.36 0)
+    (property "Reference" "C50" (id 0) (at 157.48 86.36 0)
       (effects (font (size 1.27 1.27)) (justify left))
     )
@@
   (symbol (lib_id "Device:C") (at 77.47 92.71 0) (unit 1)
     (in_bom yes) (on_board yes)
-    (property "Reference" "C45" (id 0) (at 78.74 90.1699 0)
+    (property "Reference" "C46" (id 0) (at 78.74 90.1699 0)
       (effects (font (size 1.27 1.27)) (justify left))
     )
@@
   (symbol (lib_id "Device:C") (at 38.1 77.47 0) (unit 1)
     (in_bom yes) (on_board yes)
-    (property "Reference" "C42" (id 0) (at 39.37 74.9299 0)
+    (property "Reference" "C43" (id 0) (at 39.37 74.9299 0)
       (effects (font (size 1.27 1.27)) (justify left))
     )
@@
   (symbol (lib_id "Device:C") (at 52.07 78.74 0) (unit 1)
     (in_bom yes) (on_board yes)
-    (property "Reference" "C43" (id 0) (at 53.34 76.1999 0)
+    (property "Reference" "C44" (id 0) (at 53.34 76.1999 0)
       (effects (font (size 1.27 1.27)) (justify left))
     )
@@
   (symbol (lib_id "Device:C") (at 203.2 83.82 0) (unit 1)
     (in_bom yes) (on_board yes)
-    (property "Reference" "C52" (id 0) (at 204.47 81.2799 0)
+    (property "Reference" "C53" (id 0) (at 204.47 81.2799 0)
       (effects (font (size 1.27 1.27)) (justify left))
     )
@@
   (symbol (lib_id "Device:C") (at 256.54 83.82 0) (unit 1)
     (in_bom yes) (on_board yes)
-    (property "Reference" "C57" (id 0) (at 257.81 81.28 0)
+    (property "Reference" "C58" (id 0) (at 257.81 81.28 0)
       (effects (font (size 1.27 1.27)) (justify left))
     )
@@
   (symbol (lib_id "Device:C") (at 224.79 83.82 0) (unit 1)
     (in_bom yes) (on_board yes)
-    (property "Reference" "C54" (id 0) (at 226.06 81.2799 0)
+    (property "Reference" "C55" (id 0) (at 226.06 81.2799 0)
       (effects (font (size 1.27 1.27)) (justify left))
     )
@@
   (symbol (lib_id "Device:C") (at 179.07 83.82 0) (unit 1)
     (in_bom yes) (on_board yes)
-    (property "Reference" "C50" (id 0) (at 180.34 81.2799 0)
+    (property "Reference" "C51" (id 0) (at 180.34 81.2799 0)
       (effects (font (size 1.27 1.27)) (justify left))
     )
@@
   (symbol (lib_id "Device:C") (at 214.63 83.82 0) (unit 1)
     (in_bom yes) (on_board yes)
-    (property "Reference" "C53" (id 0) (at 215.9 81.2799 0)
+    (property "Reference" "C54" (id 0) (at 215.9 81.2799 0)
       (effects (font (size 1.27 1.27)) (justify left))
     )
@@
   (symbol (lib_id "Device:C") (at 245.11 83.82 0) (unit 1)
     (in_bom yes) (on_board yes)
-    (property "Reference" "C56" (id 0) (at 246.38 81.28 0)
+    (property "Reference" "C57" (id 0) (at 246.38 81.28 0)
       (effects (font (size 1.27 1.27)) (justify left))
     )
@@
   (symbol (lib_id "Device:C") (at 68.58 90.17 0) (unit 1)
     (in_bom yes) (on_board yes)
-    (property "Reference" "C44" (id 0) (at 69.85 87.6299 0)
+    (property "Reference" "C45" (id 0) (at 69.85 87.6299 0)
       (effects (font (size 1.27 1.27)) (justify left))
     )
@@
   (symbol (lib_id "Device:C") (at 143.51 102.87 0) (unit 1)
     (in_bom yes) (on_board yes)
-    (property "Reference" "C47" (id 0) (at 144.78 100.3299 0)
+    (property "Reference" "C48" (id 0) (at 144.78 100.3299 0)
       (effects (font (size 1.27 1.27)) (justify left))
     )
@@
   (symbol (lib_id "Device:C") (at 87.63 95.25 0) (unit 1)
     (in_bom yes) (on_board yes)
-    (property "Reference" "C46" (id 0) (at 88.9 92.7099 0)
-      (effects (font (size 1.27 1.27)) (justify left))
-    )
+    (property "Reference" "C47" (id 0) (at 88.9 92.7099 0)
+      (effects (font (size 1.27 1.27)) (justify left))
+    )
