File: QuarkCncQuadDriver.kicad_sch (KiCad schematic)
At the start: 29 parts, among them J1 Screw_Terminal_01x02, J10 Screw_Terminal_01x02, J11 Screw_Terminal_01x04, J12 Screw_Terminal_01x04, J13 Screw_Terminal_01x04, J2 Conn_01x03_Male, J3 USB_B_Micro, J4 Screw_Terminal_01x02, J5 Screw_Terminal_01x02, J6 Conn_02x04_Odd_Even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

Commit message: Keyed stepper drivers. Larger input connector
Parts:
- J1: footprint Connector_Phoenix_MC:PhoenixContact_MC_1,5_2-G-3.81_1x02_P3.81mm_Horizontal -> Connector_Phoenix_MSTB:PhoenixContact_MSTBA_2,5_2-G-5,08_1x02_P5.08mm_Horizontal; LCSC C8387 -> C90074
