File: isolated_rs485.kicad_sch (KiCad schematic)
At the start: 8 parts, among them J14 Conn_01x02_Male, U26 SP3485EN-L/TR

Commit message: Keyed stepper drivers. Larger input connector
Parts:
- renumbered C58 to C59
Changed lines of the file:
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@@
   (symbol (lib_id "Device:C") (at 165.1 69.85 0) (unit 1)
     (in_bom yes) (on_board yes)
-    (property "Reference" "C58" (id 0) (at 161.29 66.6749 0)
+    (property "Reference" "C59" (id 0) (at 161.29 66.6749 0)
       (effects (font (size 1.27 1.27)) (justify left))
     )
